File: pcb/panel.kicad_pcb (KiCad board)
At the start: 2 copper layers, 81 x 131 mm, 295 parts, among them J1 CONN_04, J2 RASPBERRYPI-40-PIN-GPIO, J3 1890963, J4 1890963, J5 1890963, J6 CONN_04X2, J7 1890963, J8 1890963, J9 PI 5V, Q1 AGM60P85AP, Q2 AGM60P85AP, Q3 AGM60P85AP, Q4 2N7002, Q5 2N7002, Q6 AGM60P85AP, Q7 AGM60P85AP, Q8 2N7002, Q9 2N7002, SW1 SW_Coded_SH-7050, U1 TPS54531DDA, U2 PCA9685PW, U3 LM73100

Commit message: v2.4 as-manufactured
Parts:
- removed the C13 at (131.0, 109.2)
- removed the C13 at (131.0, 50.2)
- removed the C14 at (129.1, 49.6)
- removed the C14 at (129.1, 108.6)
- removed the D1 at (170.9, 81.8)
- removed the D1 at (170.9, 140.8)
- removed the D10 at (138.8, 72.1)
- removed the D10 at (138.8, 131.1)
- removed the D12 at (126.6, 127.8)
- removed the D12 at (126.6, 68.8)
- removed D14 (x2), D15 (x2), D27 (x2), D28 (x2): DSK34, misc:D_SOD-123F_silkpolarity
- removed the D16 at (135.0, 110.4)
- removed the D16 at (135.0, 51.4)
- removed the D19 at (140.1, 140.9)
- removed the D19 at (140.1, 81.9)
- removed the D20 at (179.2, 108.4)
- removed the D20 at (179.2, 49.4)
- removed the D25 at (141.2, 67.5)
- removed the D25 at (141.2, 126.5)
- removed the D26 at (156.2, 43.2)
- removed the D26 at (156.2, 102.2)
- removed the D29 at (123.2, 140.9)
- removed the D29 at (123.2, 81.9)
- removed the D30 at (179.2, 125.9)
- removed the D30 at (179.2, 66.9)
- removed the D31 at (138.2, 140.9)
- removed the D31 at (138.2, 81.9)
- removed the D37 at (179.2, 51.4)
- removed the D37 at (179.2, 110.4)
- removed the D38 at (173.1, 140.8)
- removed the D38 at (173.1, 81.8)
- removed the D4 at (125.1, 81.9)
- removed the D4 at (125.1, 140.9)
- removed the D5 at (179.2, 123.9)
- removed the D5 at (179.2, 64.9)
- removed the D8 at (138.8, 126.5)
- removed the D8 at (138.8, 67.5)
- removed the J7 at (180.8, 116.7)
- removed the J7 at (180.8, 57.7)
- removed the J9 at (126.1, 47.6)
- removed the J9 at (126.1, 106.6)
- removed the LOGO1 at (177.1, 66.5)
- removed the LOGO1 at (177.1, 125.5)
- removed the R1 at (170.9, 78.5)
- removed the R1 at (170.9, 137.5)
- removed the R15 at (140.2, 78.4)
- removed the R15 at (140.2, 137.4)
- removed the R19 at (135.4, 81.6)
- removed the R19 at (135.4, 140.6)
- removed the R20 at (157.6, 99.4)
- removed the R20 at (157.6, 40.4)
- removed the R21 at (138.3, 75.8)
- removed the R21 at (138.3, 134.8)
- removed the R23 at (173.1, 78.5)
- removed the R23 at (173.1, 137.5)
- removed the R9 at (123.9, 136.4)
- removed the R9 at (123.9, 77.4)
- removed the SW1 at (125.2, 117.3)
- removed the SW1 at (125.2, 58.3)
- added C13: 100uF 6.3V, Capacitor_Tantalum_SMD:CP_EIA-3528-21_Kemet-B, B.Cu at (131.0, 109.5)
- added C13: 100uF 6.3V, Capacitor_Tantalum_SMD:CP_EIA-3528-21_Kemet-B, B.Cu at (131.0, 50.5)
- added C14: 47uF, misc:C_1206_3216Metric_nosilk, F.Cu at (129.9, 108.8)
- added C14: 47uF, misc:C_1206_3216Metric_nosilk, F.Cu at (129.9, 49.8)
- added C21: 0.1uF, misc:C_0603_1608Metric_nosilk, B.Cu at (171.7, 70.2)
- added C21: 0.1uF, misc:C_0603_1608Metric_nosilk, B.Cu at (171.7, 129.2)
- added C25: 0.1uF, misc:C_0603_1608Metric_nosilk, B.Cu at (171.7, 68.7)
- added C25: 0.1uF, misc:C_0603_1608Metric_nosilk, B.Cu at (171.7, 127.7)
- added C26: 0.1uF, misc:C_0603_1608Metric_nosilk, B.Cu at (156.6, 48.6)
- added C26: 0.1uF, misc:C_0603_1608Metric_nosilk, B.Cu at (156.6, 107.7)
- added C27: 0.1uF, misc:C_0603_1608Metric_nosilk, F.Cu at (156.7, 61.0)
- added C27: 0.1uF, misc:C_0603_1608Metric_nosilk, F.Cu at (156.7, 120.0)
- added C28: 0.1uF, misc:C_0603_1608Metric_nosilk, B.Cu at (138.2, 140.5)
- added C28: 0.1uF, misc:C_0603_1608Metric_nosilk, B.Cu at (138.2, 81.5)
- added C29: 0.1uF, misc:C_0603_1608Metric_nosilk, B.Cu at (123.0, 65.0)
- added C29: 0.1uF, misc:C_0603_1608Metric_nosilk, B.Cu at (123.0, 124.0)
- added C30: 0.1uF, misc:C_0603_1608Metric_nosilk, F.Cu at (136.9, 46.0)
- added C30: 0.1uF, misc:C_0603_1608Metric_nosilk, F.Cu at (136.9, 105.0)
- added D1: SZYY0805R, misc:LED_0805_2012Metric, F.Cu at (163.6, 66.8)
- added D1: SZYY0805R, misc:LED_0805_2012Metric, F.Cu at (163.6, 125.8)
- added D10: DSK34, misc:D_SOD-123F_silkpolarity, B.Cu at (138.7, 130.8)
- added D10: DSK34, misc:D_SOD-123F_silkpolarity, B.Cu at (138.7, 71.8)
- added D12: DSK34, misc:D_SOD-123F_silkpolarity, B.Cu at (126.9, 127.8)
- added D12: DSK34, misc:D_SOD-123F_silkpolarity, B.Cu at (126.9, 68.8)
- added D16: SMBJ5.0A, misc:D_SMB_silkpolarity, B.Cu at (135.0, 51.9)
- added D16: SMBJ5.0A, misc:D_SMB_silkpolarity, B.Cu at (135.0, 110.9)
- added D19: SZYY0805R, misc:LED_0805_2012Metric, F.Cu at (140.4, 140.9)
- added D19: SZYY0805R, misc:LED_0805_2012Metric, F.Cu at (140.4, 81.9)
- added D20: SZYY0805R, misc:LED_0805_2012Metric, F.Cu at (179.2, 107.8)
- added D20: SZYY0805R, misc:LED_0805_2012Metric, F.Cu at (179.2, 48.8)
- added D25: DSK34, misc:D_SOD-123F_silkpolarity, B.Cu at (141.0, 126.3)
- added D25: DSK34, misc:D_SOD-123F_silkpolarity, B.Cu at (141.0, 67.3)
- added D26: DSK34, misc:D_SOD-123F_silkpolarity, B.Cu at (156.2, 101.6)
- added D26: DSK34, misc:D_SOD-123F_silkpolarity, B.Cu at (156.2, 42.6)
- added D29: SZYY0805YG, misc:LED_0805_2012Metric, F.Cu at (123.5, 140.9)
- added D29: SZYY0805YG, misc:LED_0805_2012Metric, F.Cu at (123.5, 81.9)
- added D30: SZYY0805YG, misc:LED_0805_2012Metric, F.Cu at (179.2, 65.8)
- added D30: SZYY0805YG, misc:LED_0805_2012Metric, F.Cu at (179.2, 124.8)
- added D31: SZYY0805YG, misc:LED_0805_2012Metric, F.Cu at (138.6, 81.9)
- added D31: SZYY0805YG, misc:LED_0805_2012Metric, F.Cu at (138.6, 140.9)
- added D37: SZYY0805YG, misc:LED_0805_2012Metric, F.Cu at (179.2, 50.8)
- added D37: SZYY0805YG, misc:LED_0805_2012Metric, F.Cu at (179.2, 109.8)
- added D38: SZYY0805YG, misc:LED_0805_2012Metric, F.Cu at (163.6, 123.8)
- added D38: SZYY0805YG, misc:LED_0805_2012Metric, F.Cu at (163.6, 64.8)
- added D39: BZT52C5V1T, misc:D_SOD-523_silkpolarity, B.Cu at (171.7, 126.1)
- added D39: BZT52C5V1T, misc:D_SOD-523_silkpolarity, B.Cu at (171.7, 67.1)
- added D4: SZYY0805R, misc:LED_0805_2012Metric, F.Cu at (125.3, 81.9)
- added D4: SZYY0805R, misc:LED_0805_2012Metric, F.Cu at (125.3, 140.9)
- added D40: DSK34, misc:D_SOD-123F_silkpolarity, B.Cu at (172.6, 65.2)
- added D40: DSK34, misc:D_SOD-123F_silkpolarity, B.Cu at (172.6, 124.2)
- added D41: SZYY0805R, misc:LED_0805_2012Metric, F.Cu at (170.7, 80.5)
- added D41: SZYY0805R, misc:LED_0805_2012Metric, F.Cu at (170.7, 139.5)
- added D42: BZT52C5V1T, misc:D_SOD-523_silkpolarity, B.Cu at (158.1, 46.0)
- added D42: BZT52C5V1T, misc:D_SOD-523_silkpolarity, B.Cu at (158.1, 105.0)
- added D43: BZT52C5V1T, misc:D_SOD-523_silkpolarity, F.Cu at (155.4, 111.5)
- added D43: BZT52C5V1T, misc:D_SOD-523_silkpolarity, F.Cu at (155.4, 52.5)
- added D44: BZT52C5V1T, misc:D_SOD-523_silkpolarity, B.Cu at (138.6, 133.8)
- added D44: BZT52C5V1T, misc:D_SOD-523_silkpolarity, B.Cu at (138.6, 74.8)
- added D45: BZT52C5V1T, misc:D_SOD-523_silkpolarity, B.Cu at (126.8, 71.8)
- added D45: BZT52C5V1T, misc:D_SOD-523_silkpolarity, B.Cu at (126.8, 130.8)
- added D5: SZYY0805R, misc:LED_0805_2012Metric, F.Cu at (179.2, 122.8)
- added D5: SZYY0805R, misc:LED_0805_2012Metric, F.Cu at (179.2, 63.8)
- added D8: DSK34, misc:D_SOD-123F_silkpolarity, B.Cu at (138.6, 67.3)
- added D8: DSK34, misc:D_SOD-123F_silkpolarity, B.Cu at (138.6, 126.3)
- added J10: 1890963, misc:Connector_Phoenix-Contact_MKDSN_1890963_P5.0_2x, F.Cu at (180.8, 72.2)
- added J10: 1890963, misc:Connector_Phoenix-Contact_MKDSN_1890963_P5.0_2x, F.Cu at (180.8, 131.2)
- added J11: ENABLE, misc:PinHeader_1x02_P2.54mm_Vertical_nosilk, F.Cu at (173.2, 81.8)
- added J11: ENABLE, misc:PinHeader_1x02_P2.54mm_Vertical_nosilk, F.Cu at (173.2, 140.8)
- added J7: 1890963, misc:Connector_Phoenix-Contact_MKDSN_1890963_P5.0_2x, F.Cu at (180.8, 57.2)
- added J7: 1890963, misc:Connector_Phoenix-Contact_MKDSN_1890963_P5.0_2x, F.Cu at (180.8, 116.2)
- added J9: PI 5V, misc:PinHeader_1x02_P2.54mm_Vertical_nosilk, F.Cu at (126.0, 47.7)
- added J9: PI 5V, misc:PinHeader_1x02_P2.54mm_Vertical_nosilk, F.Cu at (126.0, 106.7)
- added LOGO1: OSHW-Logo2_7.3x6mm_SilkScreen, Symbol:OSHW-Logo2_7.3x6mm_SilkScreen, B.Cu at (172.5, 116.3)
- added LOGO1: OSHW-Logo2_7.3x6mm_SilkScreen, Symbol:OSHW-Logo2_7.3x6mm_SilkScreen, B.Cu at (172.5, 57.3)
- added R1: 1k, Resistor_SMD:R_0603_1608Metric, B.Cu at (158.9, 69.8)
- added R1: 1k, Resistor_SMD:R_0603_1608Metric, B.Cu at (158.9, 128.8)
- added R15: 1k, Resistor_SMD:R_0603_1608Metric, B.Cu at (140.2, 137.5)
- added R15: 1k, Resistor_SMD:R_0603_1608Metric, B.Cu at (140.2, 78.5)
- added R19: 1k, Resistor_SMD:R_0603_1608Metric, B.Cu at (135.8, 81.6)
- added R19: 1k, Resistor_SMD:R_0603_1608Metric, B.Cu at (135.8, 140.6)
- added R20: 1k, Resistor_SMD:R_0603_1608Metric, B.Cu at (157.7, 98.8)
- added R20: 1k, Resistor_SMD:R_0603_1608Metric, B.Cu at (157.7, 39.9)
- added R21: 10k, Resistor_SMD:R_0603_1608Metric, B.Cu at (141.8, 78.5)
- added R21: 10k, Resistor_SMD:R_0603_1608Metric, B.Cu at (141.8, 137.5)
- added R23: 1k, Resistor_SMD:R_0603_1608Metric, B.Cu at (158.9, 67.6)
- added R23: 1k, Resistor_SMD:R_0603_1608Metric, B.Cu at (158.9, 126.6)
- added R47: 10k, Resistor_SMD:R_0603_1608Metric, B.Cu at (171.7, 71.8)
- added R47: 10k, Resistor_SMD:R_0603_1608Metric, B.Cu at (171.7, 130.8)
- added R48: 1k, Resistor_SMD:R_0603_1608Metric, B.Cu at (175.9, 72.0)
- added R48: 1k, Resistor_SMD:R_0603_1608Metric, B.Cu at (175.9, 131.1)
- added R49: 1k, Resistor_SMD:R_0603_1608Metric, B.Cu at (172.9, 73.3)
- added R49: 1k, Resistor_SMD:R_0603_1608Metric, B.Cu at (172.9, 132.3)
- added R50: 10k, Resistor_SMD:R_0603_1608Metric, B.Cu at (157.8, 44.5)
- added R50: 10k, Resistor_SMD:R_0603_1608Metric, B.Cu at (157.8, 103.5)
- added R51: 10k, Resistor_SMD:R_0603_1608Metric, B.Cu at (156.9, 118.2)
- added R51: 10k, Resistor_SMD:R_0603_1608Metric, B.Cu at (156.9, 59.2)
- added R52: 10k, Resistor_SMD:R_0603_1608Metric, B.Cu at (138.4, 76.2)
- added R52: 10k, Resistor_SMD:R_0603_1608Metric, B.Cu at (138.4, 135.2)
- added R53: 10k, Resistor_SMD:R_0603_1608Metric, B.Cu at (126.5, 132.3)
- added R53: 10k, Resistor_SMD:R_0603_1608Metric, B.Cu at (126.5, 73.3)
- added R54: 470, Resistor_SMD:R_0603_1608Metric, B.Cu at (174.6, 106.2)
- added R54: 470, Resistor_SMD:R_0603_1608Metric, B.Cu at (174.6, 47.2)
- added R55: 470, Resistor_SMD:R_0603_1608Metric, B.Cu at (171.3, 136.8)
- added R55: 470, Resistor_SMD:R_0603_1608Metric, B.Cu at (171.3, 77.8)
- added R56: 470, Resistor_SMD:R_0603_1608Metric, B.Cu at (174.6, 121.6)
- added R56: 470, Resistor_SMD:R_0603_1608Metric, B.Cu at (174.6, 62.6)
- added R57: 470, Resistor_SMD:R_0603_1608Metric, B.Cu at (138.7, 78.5)
- added R57: 470, Resistor_SMD:R_0603_1608Metric, B.Cu at (138.7, 137.5)
- added R58: 470, Resistor_SMD:R_0603_1608Metric, B.Cu at (123.5, 78.6)
- added R58: 470, Resistor_SMD:R_0603_1608Metric, B.Cu at (123.5, 137.6)
- added R9: 1k, Resistor_SMD:R_0603_1608Metric, B.Cu at (126.5, 74.8)
- added R9: 1k, Resistor_SMD:R_0603_1608Metric, B.Cu at (126.5, 133.8)
- added SW1: SW_Coded_SH-7050, misc:Diptronics-Rotary-Switch-R7M3-16RA-V, F.Cu at (125.4, 117.3)
- added SW1: SW_Coded_SH-7050, misc:Diptronics-Rotary-Switch-R7M3-16RA-V, F.Cu at (125.4, 58.3)
- added U4: 74LVC1G08, Package_TO_SOT_SMD:SOT-353_SC-70-5, B.Cu at (140.7, 140.4)
- added U4: 74LVC1G08, Package_TO_SOT_SMD:SOT-353_SC-70-5, B.Cu at (140.7, 81.5)
- added U5: 74LVC1G08, Package_TO_SOT_SMD:SOT-353_SC-70-5, B.Cu at (125.3, 64.8)
- added U5: 74LVC1G08, Package_TO_SOT_SMD:SOT-353_SC-70-5, B.Cu at (125.3, 123.8)
- added U6: 74LVC1G08, Package_TO_SOT_SMD:SOT-353_SC-70-5, B.Cu at (156.8, 120.5)
- added U6: 74LVC1G08, Package_TO_SOT_SMD:SOT-353_SC-70-5, B.Cu at (156.8, 61.5)
- added U7: 74LVC1G08, Package_TO_SOT_SMD:SOT-353_SC-70-5, B.Cu at (158.8, 107.4)
- added U7: 74LVC1G08, Package_TO_SOT_SMD:SOT-353_SC-70-5, B.Cu at (158.8, 48.4)
- added U8: 74LVC1G08, Package_TO_SOT_SMD:SOT-353_SC-70-5, B.Cu at (171.7, 134.6)
- added U8: 74LVC1G08, Package_TO_SOT_SMD:SOT-353_SC-70-5, B.Cu at (171.7, 75.5)
- added U9: AZ1117-3.3, Package_TO_SOT_SMD:SOT-23, B.Cu at (132.7, 105.3)
- added U9: AZ1117-3.3, Package_TO_SOT_SMD:SOT-23, B.Cu at (132.7, 46.3)
- D17 (x2), D18 (x2), D2 (x2), D3 (x2), D6 (x2): value BZT52C9V1TQ-7-F -> BZT52C5V1T
- R46 (x2): value 165k -> 360k
- turned D6 to 180 degrees (x2)
- turned R16 to 0 degrees (x2)
Connections:
- net Board_0-Net-(D12-A) renamed Board_0-Net-(Q4-G)
- net Board_0-Net-(D26-A) renamed Board_0-Net-(Q9-G)
- net Board_0-unconnected-(U3-DVDT-Pad7)_0 renamed Board_0-unconnected-(U3-DVDT-Pad7)
- net Board_1-Net-(D12-A) renamed Board_1-Net-(Q4-G)
- net Board_1-Net-(D26-A) renamed Board_1-Net-(Q9-G)
- net Board_1-unconnected-(U3-DVDT-Pad7)_0 renamed Board_1-unconnected-(U3-DVDT-Pad7)
- J2 pad 1: Board_0-+3V3 -> Board_0-unconnected-(J2-3.3V-Pad1)
- J2 pad 1: Board_1-+3V3 -> Board_1-unconnected-(J2-3.3V-Pad1)
- Q5 pad 1: Board_0-Net-(D13-A) -> Board_0-Net-(Q5-G)
- Q5 pad 1: Board_1-Net-(D13-A) -> Board_1-Net-(Q5-G)
- Q8 pad 1: Board_0-Net-(D25-A) -> Board_0-Net-(Q8-G)
- Q8 pad 1: Board_1-Net-(D25-A) -> Board_1-Net-(Q8-G)
- R12 pad 2: Board_1-Net-(D13-A) -> Board_1-Net-(Q5-G)
- R12 pad 2: Board_0-Net-(D13-A) -> Board_0-Net-(Q5-G)
- R16 pad 1: Board_0-Net-(D20-A) -> Board_0-/M4_D
- R16 pad 2: Board_0-/M4_D -> Board_0-Net-(D20-A)
- R16 pad 1: Board_1-Net-(D20-A) -> Board_1-/M4_D
- R16 pad 2: Board_1-/M4_D -> Board_1-Net-(D20-A)
Routing:
- net Board_1-ENABLE: track 0.00 -> 126.5 mm, vias 0 -> 6
- net Board_0-ENABLE: track 0.00 -> 126.5 mm, vias 0 -> 6
- net Board_1-+3V3: track 81.6 -> 194.7 mm, vias 3 -> 11
- net Board_0-+3V3: track 81.6 -> 194.7 mm, vias 3 -> 11
- net Board_1-VIN: track 29.9 -> 0.00 mm, vias 2 -> 0
- net Board_0-VIN: track 29.9 -> 0.00 mm, vias 2 -> 0
- net Board_1-Net-(D1-K): track 29.5 -> 4.29 mm
- net Board_0-Net-(D1-K): track 29.5 -> 4.29 mm
- net Board_1-Net-(D13-A): track 31.9 -> 11.1 mm, vias 2 -> 1
- net Board_0-Net-(D13-A): track 31.9 -> 11.1 mm, vias 2 -> 1
- net Board_0-Net-(Q5-G): track 0.00 -> 17.7 mm
- net Board_1-Net-(Q5-G): track 0.00 -> 17.7 mm
- net Board_1-Net-(J10-Pin_2): track 0.00 -> 12.4 mm
- net Board_0-Net-(J10-Pin_2): track 0.00 -> 12.4 mm
- net Board_0-GND: track 46.7 -> 58.5 mm, vias 51 -> 59
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Other:
- board text added: "#1 ON"
- board text added: "#2 ON"
- board text added: "#4 ON"
- board text added: "2024-06-08"
- board text added: "EN"
- board text added: "EN +"
- board text added: "INPUT 7V-26V MAX 7A MAX 2A PER OUTPUT, SWITCHED +VE OUTPUT CONTROL VIA: 1. PI GPIO (JUMPER TO LEFT POS.) 2. PCA9685 PWM CTRL. (RIGHT) 3. DIRECT 3V-26V SIGNAL (CTR)"
- board text added: "OUTPUT ENABLE"
- board text added: "owl-driver-board-v2.4"
- board text added: "v2.4"
- board text removed: "2024-03-16"
- board text removed: "7-26V"
- board text removed: "INPUT 7V-26V MAX 7A MAX 2A PER OUTPUT, SWITCHED +VE OUTPUT CONTROL VIA: 1. PI GPIO (JUMPER TO LEFT POS.) 2. PCA9685 PWM CTRL. (RIGHT POS.) 3. DIRECT 3V-26V SIGNAL (CTR. PIN)"
- board text removed: "github.com/geezacoleman/ owl-driver-board"
- board text removed: "owl-driver-board-v2.3"
- board text removed: "v2.0"
- board text removed: "v2.3 202406"
