File: owl-driver-board-16/output_chain.kicad_sch (KiCad schematic)
At the start: 20 parts, among them J4 1890963, Q2 AGM60P85AP, Q4 2N7002, U5 74LVC1G08

Commit message: add a 16-way version
Add a 16-way version of the HAT. Drop the PWM controller to focus on
GPIO control of 16 outputs, with output enable/e-stop, and keeping the
25W Pi power supply.

This version (v1.0) has a small bug in the panel, fixed in v1.1.
Parts:
- C29: value 0.1uF -> 10uF; footprint misc:C_0603_1608Metric_nosilk -> misc:C_1206_3216Metric_nosilk; LCSC C14663 -> C13585; Part (none) -> CL31A106KBHNNNE
- D29: value SZYY0805YG -> KT-0805G; LCSC C434435 -> C2297; Part (none) -> KT-0805G
- D4: value SZYY0805R -> KT-0805Y; LCSC C434431 -> C2296; Part (none) -> KT-0805Y
Connections:
- net OUTPUT+: now reaches D4.1 (K), F2.2, J4.1 (Pin_1)
- net M1_D renamed DRAIN
- net M1_G renamed GATE
Other:
- note added: "SOURCE"
- note removed: "M1_S"
Changed lines of the file:
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@@
 	(generator_version "9.0")
 	(paper "A4")
-	(text "M1_S"
+	(text "SOURCE"
 		(exclude_from_sim no)
-		(at 186.69 72.39 90)
+		(at 186.69 69.85 90)
 		(effects
 			(font
@@
 		)
 	)
-	(label "M1_G"
+	(label "OUTPUT+"
+		(at 226.06 90.17 0)
+		(effects
+			(font
+				(size 1.27 1.27)
+			)
+			(justify left bottom)
+		)
+	)
+	(label "GATE"
 		(at 176.53 83.82 180)
 		(effects
@@
 		)
 	)
-	(label "M1_D"
+	(label "DRAIN"
 		(at 187.96 90.17 0)
 		(effects
@@
 			)
 		)
-		(property "Value" "SZYY0805YG"
+		(property "Value" "KT-0805G"
 			(at 154.051 117.1015 90)
 			(effects
@@
 			)
 		)
-		(property "Datasheet" "https://datasheet.lcsc.com/lcsc/1912111437_Yongyu-Photoelectric-SZYY0805YG_C434435.pdf"
+		(property "Datasheet" "https://jlcpcb.com/api/file/downloadByFileSystemAccessId/8550724011370958848"
 			(at 152.4 119.38 0)
 			(effects
@@
 			)
 		)
-		(property "LCSC" "C434435"
+		(property "LCSC" "C2297"
 			(at 152.4 119.38 0)
 			(effects
@@
 			)
 		)
+		(property "Part" "KT-0805G"
+			(at 152.4 119.38 0)
+			(effects
+				(font
+					(size 1.27 1.27)
+				)
+			)
+		)
 		(pin "1"
 		)
@@
 			)
 		)
-		(property "Value" "SZYY0805R"
+		(property "Value" "KT-0805Y"
 			(at 214.8915 79.629 90)
 			(effects
@@
 			)
 		)
-		(property "LCSC" "C434431"
+		(property "LCSC" "C2296"
 			(at 217.17 81.28 0)
 			(effects
@@
 			)
 		)
+		(property "Part" "KT-0805Y"
+			(at 217.17 81.28 0)
+			(effects
+				(font
+					(size 1.27 1.27)
+				)
+			)
+		)
 		(pin "1"
 		)
@@
 			)
 		)
-		(property "Value" "0.1uF"
+		(property "Value" "10uF"
 			(at 125.73 91.4399 0)
 			(effects
@@
 			)
 		)
-		(property "Footprint" "misc:C_0603_1608Metric_nosilk"
+		(property "Footprint" "misc:C_1206_3216Metric_nosilk"
 			(at 122.8852 93.98 0)
 			(effects
@@
 			)
 		)
-		(property "Datasheet" "https://datasheet.lcsc.com/lcsc/1811021431_Samsung-Electro-Mechanics-CL10B104KB8NNNC_C1591.pdf"
+		(property "Datasheet" ""
 			(at 121.92 90.17 0)
 			(effects
@@
 			)
 		)
-		(property "LCSC" "C14663"
+		(property "LCSC" "C13585"
+			(at 121.92 90.17 0)
+			(effects
+				(font
+					(size 1.27 1.27)
+				)
+				(hide yes)
+			)
+		)
+		(property "Part" "CL31A106KBHNNNE"
 			(at 121.92 90.17 0)
 			(effects
